File: knx-mikrobus-board/knx-mikrobus-board.kicad_pcb (KiCad board)
At the start: 2 copper layers, 25.4 x 42.9 mm, 30 parts, among them J1 mikroBUS_L, J2 mikroBUS_R, J3 KNX+, J4 KNX-, U1 NCN5130, X1 16MHz

Commit message: knx: add ground plane
Connections:
- U1 pad 41: unconnected-(U1-Pad41) -> /knx-logic/GND
Routing:
- net /knx-logic/GND: track 157.6 -> 144.9 mm
- added copper zone on B.Cu, net /knx-logic/GND
- added copper zone on F.Cu, net /knx-logic/GND
