File: i2c-spi-oled-mikrobus-board/i2c-spi-oled-mikrobus-board.kicad_sch (KiCad schematic)
At the start: 10 parts, among them J1 mikroBUS_L, J2 mikroBUS_R, J3 Conn_02x08_Odd_Even, U1 SC18IS606PW, U2 PCA9557PW

Commit message: i2c-spi-oled: also connect the R/~W pin
the display doesn't need it (it will be held to GND) but we might reuse
this board for other SPI components
Connections:
- net GND: no longer J3.1 (Pin_1)
- net D_R_~{W}: now reaches U2.10 (IO3)
- net D_R_~{W}: now also J3.1 (Pin_1)
- no-connect marks 22 -> 21
Changed lines of the file:
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@@
   (no_connect (at 101.6 149.86))
   (no_connect (at 73.66 110.49))
-  (no_connect (at 73.66 105.41))
   (bus_entry (at 44.45 116.84) (size 2.54 -2.54)
     (stroke (width 0) (type default) (color 0 0 0 0))
@@
     (stroke (width 0) (type default) (color 0 0 0 0))
   )
+  (bus_entry (at 92.71 102.87) (size -2.54 2.54)
+    (stroke (width 0) (type default) (color 0 0 0 0))
+  )
   (bus_entry (at 156.21 170.18) (size -2.54 2.54)
     (stroke (width 0) (type default) (color 0 0 0 0))
@@
     (stroke (width 0) (type default) (color 0 0 0 0))
   )
+  (wire (pts (xy 73.66 105.41) (xy 90.17 105.41))
+    (stroke (width 0) (type default) (color 0 0 0 0))
+  )
   (wire (pts (xy 124.46 68.58) (xy 124.46 74.93))
     (stroke (width 0) (type default) (color 0 0 0 0))
@@
     (stroke (width 0) (type default) (color 0 0 0 0))
   )
+  (bus (pts (xy 92.71 102.87) (xy 92.71 104.14))
+    (stroke (width 0) (type default) (color 0 0 0 0))
+  )
   (bus (pts (xy 16.51 113.03) (xy 16.51 110.49))
     (stroke (width 0) (type default) (color 0 0 0 0))
@@
     (stroke (width 0) (type default) (color 0 0 0 0))
   )
-  (bus (pts (xy 92.71 101.6) (xy 92.71 104.14))
+  (bus (pts (xy 92.71 101.6) (xy 92.71 102.87))
     (stroke (width 0) (type default) (color 0 0 0 0))
   )
@@
     (effects (font (size 1.27 1.27)) (justify left bottom))
   )
+  (label "D_R_~{W}" (at 73.66 105.41 0)
+    (effects (font (size 1.27 1.27)) (justify left bottom))
+  )
   (label "{ALLBUS}" (at 66.04 144.78 180)
     (effects (font (size 1.27 1.27)) (justify right bottom))
@@
     (effects (font (size 1.27 1.27)) (justify right bottom))
   )
-  (label "GND" (at 106.68 68.58 270)
-    (effects (font (size 1.27 1.27)) (justify right bottom))
-  )
+  (label "D_R_~{W}" (at 106.68 68.58 270)
+    (effects (font (size 1.27 1.27)) (justify right bottom))
+  )

Commit message: i2c-spi-oled: put ~RST signal on port expander too
Parts:
- J3: LCSC (none) -> C5338669
- JP1: now left out of the parts list
- R1: LCSC (none) -> C23179
- U1: LCSC (none) -> C5190384
- U2: LCSC (none) -> C141380
Connections:
- net ~{RST}: no longer J3.3 (Pin_3)
- net D_~{RST}: now reaches U2.11 (IO4)
- net D_~{RST}: now also J3.3 (Pin_3)
- no-connect marks 21 -> 20
